File: NonSplitKyria/NonSplitKyria.kicad_pcb (KiCad board)
At the start: 2 copper layers, 15.2 x 6.3 mm, 104 parts, among them J1 USB2_C_Receptacle, SW1 Reset, U1 ATmega32U4-AU, Y1 16MHz

Commit message: Route Diodes
Parts:
- moved F1 4.36 mm to (170.9, 23.8), turned to -90 degrees
- moved R3 3.35 mm to (173.2, 20.1)
- moved R2 3.34 mm to (178.2, 20.1)
- moved J1 3.33 mm to (175.7, 9.69)
- moved R4 3.33 mm to (174.4, 23.8)
- moved R5 3.33 mm to (176.6, 23.8)
- moved C3 2.39 mm to (172.2, 49.0)
- moved C2 2.39 mm to (184.8, 43.8)
- moved C4 2.39 mm to (167.3, 36.5)
- moved C5 2.39 mm to (184.0, 32.4)
- moved R6 2.39 mm to (181.3, 49.1)
- moved U1 2.39 mm to (176.4, 39.7)
- moved Y1 2.39 mm to (167.2, 39.4)
- moved C1 2.39 mm to (175.2, 30.4), turned to 180 degrees
- moved R1 2.39 mm to (167.3, 34.3)
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- renumbered K_42 to K_41, K_41 to K_42
Connections:
- K_41 pad 1: col7 -> col6
- K_41 pad 2: Net-(D42-Pad2) -> Net-(D41-Pad2)
- K_42 pad 1: col6 -> col7
- K_42 pad 2: Net-(D41-Pad2) -> Net-(D42-Pad2)
Routing:
- net Net-(D12-Pad2): track 0.00 -> 148.6 mm
- net Net-(D1-Pad2): track 0.00 -> 144.6 mm
- net Net-(D24-Pad2): track 0.00 -> 144.5 mm
- net Net-(D36-Pad2): track 0.00 -> 141.3 mm
- net Net-(D13-Pad2): track 0.00 -> 140.6 mm
- net Net-(D25-Pad2): track 0.00 -> 138.0 mm
- net Net-(D11-Pad2): track 0.00 -> 132.2 mm
- net Net-(D2-Pad2): track 0.00 -> 129.2 mm
- net Net-(D23-Pad2): track 0.00 -> 127.8 mm
- net Net-(D10-Pad2): track 0.00 -> 126.4 mm
- net Net-(D35-Pad2): track 0.00 -> 124.4 mm
- net Net-(D14-Pad2): track 0.00 -> 124.2 mm
- net Net-(D3-Pad2): track 0.00 -> 123.1 mm
- net Net-(D26-Pad2): track 0.00 -> 121.8 mm
- net Net-(D22-Pad2): track 0.00 -> 121.2 mm
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- added copper zone on B.Cu, net GND
- added copper zone on F.Cu, net GND
Other:
- board size 15.2 x 6.3 mm -> 323.9 x 95.1 mm
- net class PWR added: clearance 0.2, trace_width 0.381, via_dia 0.8, via_drill 0.4

Commit message: Route MCU rows + cols
Connections:
- U1 pad 19: Net-(U1-Pad19) -> col0
- U1 pad 20: Net-(U1-Pad20) -> col1
- U1 pad 21: Net-(U1-Pad21) -> col2
- U1 pad 22: Net-(U1-Pad22) -> col3
- U1 pad 25: Net-(U1-Pad25) -> col4
- U1 pad 26: Net-(U1-Pad26) -> col5
- U1 pad 27: Net-(U1-Pad27) -> row1
- U1 pad 28: Net-(U1-Pad28) -> row3
- U1 pad 29: Net-(U1-Pad29) -> row2
- U1 pad 30: Net-(U1-Pad30) -> row0
- U1 pad 31: Net-(U1-Pad31) -> col6
- U1 pad 32: Net-(U1-Pad32) -> col7
- U1 pad 37: Net-(U1-Pad37) -> col8
- U1 pad 38: Net-(U1-Pad38) -> col9
- U1 pad 39: Net-(U1-Pad39) -> col10
- U1 pad 40: Net-(U1-Pad40) -> col11
Routing:
- net col11: track 38.1 -> 230.0 mm, vias 0 -> 1
- net col0: track 38.1 -> 224.8 mm
- net col10: track 38.1 -> 210.3 mm, vias 0 -> 1
- net col1: track 38.1 -> 205.9 mm, vias 0 -> 1
- net col2: track 61.1 -> 206.2 mm
- net col9: track 61.1 -> 201.6 mm
- net col3: track 65.9 -> 189.0 mm
- net col8: track 65.9 -> 180.8 mm
- net col4: track 63.9 -> 176.9 mm
- net col7: track 65.8 -> 165.9 mm
- net col5: track 69.2 -> 163.5 mm
- net col6: track 72.6 -> 150.8 mm
- net row3: track 27.0 -> 65.8 mm
- net row2: track 39.7 -> 72.7 mm, vias 0 -> 2
- net row1: track 39.7 -> 64.1 mm, vias 0 -> 2
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Other:
- outline, holes or cut-outs redrawn

Commit message: Add Silkscreen art
Parts:
- added G***: LOGO, Local_Project:Lemur70mm, B.Cu at (176.4, 54.8)
- added REF**: WEEE-Logo_8.4x12mm_SilkScreen, Symbol:WEEE-Logo_8.4x12mm_SilkScreen, B.Cu at (205.1, 95.3)
Routing:
- net col2: track 206.2 -> 205.5 mm
- net GND: vias 19 -> 18

Commit message: Add Gerbers
Parts:
- added REF**: Symbol_Attention_CopperTop_Big, Symbol:Symbol_Attention_CopperTop_Big, F.Cu at (206.2, 32.7)
- added REF**: Symbol_Attention_CopperTop_Big, Symbol:Symbol_Attention_CopperTop_Big, F.Cu at (144.5, 32.5)
- added REF**: Symbol_Attention_CopperTop_Big, Symbol:Symbol_Attention_CopperTop_Big, F.Cu at (144.5, 23.0)
- added REF**: Symbol_Attention_CopperTop_Big, Symbol:Symbol_Attention_CopperTop_Big, F.Cu at (206.4, 23.0)
- moved G*** 0.20 mm to (176.2, 54.8)
Other:
- board text added: "Designed by swiftrax"
- board text added: "UnSplit"
